Commit message: removing realsense mesh dependency

File: covid_slam/models/d435_kinect/d435_kinect.xacro (robot description, xacro)
@@ -45,6 +45,5 @@
         <geometry>
           <!-- <box size="${d435_cam_width} ${d435_cam_height} ${d435_cam_depth}"/> -->
-          <mesh filename="package://realsense2_description/meshes/d435.dae" />
-          <!--<mesh filename="package://realsense2_description/meshes/d435/d435.dae" />-->
+          <mesh filename="package://covid_slam/models/d435_kinect/d435.dae" />
         </geometry>
         <material name="${name}_aluminum"/>

Commit message: laptop codebase

File: covid_slam/models/d435_kinect/d435_kinect.xacro (robot description, xacro)
@@ -45,5 +45,6 @@
         <geometry>
           <!-- <box size="${d435_cam_width} ${d435_cam_height} ${d435_cam_depth}"/> -->
-          <mesh filename="package://covid_slam/models/d435_kinect/d435.dae" />
+          <mesh filename="package://realsense2_description/meshes/d435.dae" />
+          <!--<mesh filename="package://realsense2_description/meshes/d435/d435.dae" />-->
         </geometry>
         <material name="${name}_aluminum"/>

Commit message: improving some compatability between real and sim files

File: covid_slam/models/d435_kinect/d435_kinect.xacro (robot description, xacro)
@@ -8,5 +8,5 @@
 <robot name="d435_kinect" xmlns:xacro="http://ros.org/wiki/xacro">
   <!--File includes-->
-  <xacro:macro name="sensor_d435_kinect" params="name:=camera topics_ns:=camera parent *origin">
+  <xacro:macro name="sensor_d435_kinect" params="name:=d435i topics_ns:=camera parent *origin">
     <xacro:property name="M_PI" value="3.1415926535897931" />
     <!-- The following values are approximate, and the camera node

Commit message: alligned simulation with the real thing

File: covid_slam/models/d435_kinect/d435_kinect.xacro (robot description, xacro)
@@ -8,5 +8,5 @@
 <robot name="d435_kinect" xmlns:xacro="http://ros.org/wiki/xacro">
   <!--File includes-->
-  <xacro:macro name="sensor_d435_kinect" params="name:=d435i topics_ns:=camera parent *origin">
+  <xacro:macro name="sensor_d435_kinect" params="name:=d435i topics_ns:=d435i parent *origin">
     <xacro:property name="M_PI" value="3.1415926535897931" />
     <!-- The following values are approximate, and the camera node

File: covid_slam/models/d435_t265/d435_t265.xacro (robot description, xacro)
@@ -1,7 +1,15 @@
 <?xml version="1.0"?>
-<robot name="d435_t265" xmlns:xacro="http://ros.org/wiki/xacro">
-  <xacro:include filename="$(find realsense2_description)/urdf/_d435.urdf.xacro"/>
-  <link name="base_link" />
-  <xacro:sensor_d435 parent="base_link" use_nominal_extrinsics="$(arg use_nominal_extrinsics)">
-  <xacro:sensor_d435>
+<root name="d435_t265" xmlns:xacro="http://ros.org/wiki/xacro">
+  <xacro:include filename="$(find covid_slam)/models/d435_kinect/d435_kinect.xacro"/>
+  <xacro:sensor_d435_kinect parent="base_link">
+      <origin xyz="0.15 0 0" rpy="0 0 0"/>
+  </xacro:sensor_d435_kinect>
+  <link name="t265_odom_frame"/>
+  <link name="t265_link"/>
+  <joint name="t265_joint" type="fixed">
+    <origin xyz="-0.15 0 .05" rpy="0 0 0"/>
+    <parent link="t265_pose_frame"/>
+    <child link="base_link"/>
+  </joint>
+  <link>
 </robot>
