Commit message: assembled all parts under quad.launch

File: covid_slam/models/quad/quad.xacro (robot description, xacro)
@@ -6,15 +6,29 @@
       <geometry>
           <mesh filename="package://covid_slam/models/quad/iris.stl"
-                scale="1 1 1"/>
+                scale="1.2 1.2 1.2"/>
       </geometry>
     </visual>
   </link>
+  <link name="t265_pose_frame"/>
   <joint name="t265_joint" type="fixed">
-    <origin xyz="0.15 -.05 0" rpy="0 0 0"/>
-    <parent link="base_link"/>
-    <child link="t265_pose_frame"/>
+    <origin xyz="-0.15 0 .05" rpy="0 0 0"/>
+    <parent link="t265_pose_frame"/>
+    <child link="base_link"/>
   </joint>
-  <!--xacro:sensor_d435_kinect parent="base_link">
-      <origin xyz="0.15 0 0" rpy="0 0 0"/>
-  </xacro:sensor_d435_kinect-->
+    <xacro:property name="d435_cam_depth_py" value="0.0175"/>
+    <xacro:property name="d435_cam_mount_from_center_offset" value="0.0149"/>
+    <xacro:property name="M_PI" value="3.1415926535897931" />
+  <link name="d435i_link">
+    <visual>
+      <origin xyz="${d435_cam_mount_from_center_offset} ${-d435_cam_depth_py} 0" rpy="${M_PI/2} 0 ${M_PI/2}"/>
+      <geometry>
+        <mesh filename="package://covid_slam/models/d435_kinect/d435.dae" />
+      </geometry>
+    </visual>
+  </link>
+  <joint name="t265_to_d435i" type="fixed">
+    <origin xyz="0 .02 0" rpy="0 0 0"/>
+    <parent link="t265_pose_frame"/>
+    <child link="d435i_link"/>
+  </joint>
 </robot>

Commit message: quad changes to verify in sim

File: covid_slam/models/quad/quad.xacro (robot description, xacro)
@@ -12,5 +12,5 @@
   <link name="t265_pose_frame"/>
   <joint name="t265_joint" type="fixed">
-    <origin xyz="-0.15 0 .05" rpy="0 0 0"/>
+    <origin xyz="-0.1 0 .06" rpy="0 0 0"/>
     <parent link="t265_pose_frame"/>
     <child link="base_link"/>

Commit message: changes from sim (critical mode, octomap)

File: covid_slam/models/quad/quad.xacro (robot description, xacro)
@@ -10,4 +10,11 @@
     </visual>
   </link>
+  <!--link name="t265_odom_frame"/>
+  <link name="map"/>
+  <joint name="t265_is_map" type="fixed">
+    <origin xyz="0 0 0" rpy="0 0 0"/>
+    <parent link="map"/>
+    <child link="t265_odom_frame"/>
+  </joint-->
   <link name="t265_pose_frame"/>
   <joint name="t265_joint" type="fixed">
